File: ParaPRZEKAZNIK.kicad_pcb (KiCad board)
At the start: 2 copper layers, 75 x 50 mm, 79 parts, among them J1 PT1000, J10 Screw_Terminal_01x03, J2 5556416-1 TE Connectivity, J3 UC_CONTROL, J4 MAIN_CONTROL, J5 PROG, J6 Screw_Terminal_01x03, J7 Screw_Terminal_01x03, J8 Screw_Terminal_01x03, J9 Screw_Terminal_01x03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

Commit message: partially routed
Connections:
- C13 pad 2: +12V -> +BATT
- C14 pad 1: /+12V_F -> +12V
- D1 pad 1: +12V -> +BATT
- L5 pad 1: +12V -> +BATT
- L5 pad 2: /+12V_F -> +12V
- U1 pad 5: /F+ -> unconnected-(U1-FORCE+-Pad5)
- U5 pad 3: /+12V_F -> +12V
Routing:
- net +12V: track 0.00 -> 153.1 mm, vias 0 -> 3
- net GND: track 0.00 -> 135.0 mm, vias 0 -> 7
- net +3V3: track 0.00 -> 72.5 mm, vias 0 -> 2
- net /CONTROL_SIG: track 0.00 -> 35.9 mm, vias 0 -> 1
- net Net-(D3-A1): track 0.00 -> 29.8 mm, vias 0 -> 1
- net /BASE_R5: track 0.00 -> 29.0 mm, vias 0 -> 2
- net /R1: track 0.00 -> 26.1 mm, vias 0 -> 2
- net /R4: track 0.00 -> 25.0 mm, vias 0 -> 2
- net Net-(D14-A): track 0.00 -> 24.9 mm, vias 0 -> 1
- net /R3: track 0.00 -> 20.6 mm, vias 0 -> 2
- net /R2: track 0.00 -> 19.6 mm, vias 0 -> 2
- net Net-(SW1B-C): track 0.00 -> 18.6 mm, vias 0 -> 1
- net Net-(D13-A): track 0.00 -> 18.3 mm, vias 0 -> 1
- net Net-(D10-A): track 0.00 -> 17.5 mm, vias 0 -> 2
- net /RELAYS_CTRL: track 0.00 -> 17.0 mm
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Other:
- board text added: "ParaPRZEKAZNIK RevA Mateusz Lubecki, Bielsko-Biala 2025"
- board text added: "RS232 Cisco style"

Commit message: done and exported
Parts:
- added R14: R, Resistor_SMD:R_0805_2012Metric_Pad1.20x1.40mm_HandSolder, F.Cu at (50.3, 53.6)
- added R15: 20k, Resistor_SMD:R_0805_2012Metric_Pad1.20x1.40mm_HandSolder, B.Cu at (69.3, 77.1)
- added R16: 120, Resistor_SMD:R_0805_2012Metric_Pad1.20x1.40mm_HandSolder, B.Cu at (79.6, 75.8)
- RN1: value 1k -> 10k
- RN2: value 10k -> 1k
- moved C11 2.81 mm to (80.5, 69.3)
- moved R7 2.55 mm to (80.5, 67.1)
- moved R9 2.55 mm to (80.5, 61.0)
- moved R8 2.54 mm to (80.3, 64.0)
- moved L5 2.09 mm to (80.3, 75.7), turned to 0 degrees
- moved D3 1.80 mm to (80.5, 72.4)
- moved C9 1.52 mm to (59.9, 70.1)
- moved R1 1.52 mm to (50.3, 78.7)
- moved R12 1.52 mm to (61.0, 73.2)
- moved C15 1.40 mm to (54.4, 54.0)
- moved R5 1.27 mm to (58.9, 65.8)
- moved R6 1.27 mm to (61.0, 65.8)
- moved C13 1.05 mm to (80.5, 78.7)
- moved SW1 1.02 mm to (86.9, 58.5)
- moved U2 1.02 mm to (57.9, 58.9)
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Connections:
- U1 pad 1: unconnected-(U1-BIAS-Pad1) -> Net-(U1-BIAS)
- U1 pad 2: unconnected-(U1-REFIN+-Pad2) -> Net-(U1-BIAS)
- U1 pad 3: unconnected-(U1-REFIN--Pad3) -> Net-(U1-ISENSOR)
- U1 pad 4: unconnected-(U1-ISENSOR-Pad4) -> Net-(U1-ISENSOR)
- U1 pad 5: unconnected-(U1-FORCE+-Pad5) -> /F+
- U1 pad 6: unconnected-(U1-FORCE2-Pad6) -> GND
Routing:
- net GND: track 135.0 -> 404.1 mm, vias 7 -> 32
- net +3V3: track 72.5 -> 172.3 mm, vias 2 -> 8
- net 485B: track 0.00 -> 51.5 mm, vias 0 -> 2
- net /R1: track 26.1 -> 73.4 mm, vias 2 -> 5
- net /R2: track 19.6 -> 63.4 mm, vias 2 -> 5
- net 485A: track 0.00 -> 41.8 mm, vias 0 -> 4
- net /R3: track 20.6 -> 62.1 mm, vias 2 -> 3
- net /R4: track 25.0 -> 65.1 mm, vias 2 -> 3
- net /BASE_R1: track 4.33 -> 42.2 mm, vias 1 -> 4
- net MICRO_CTRL: track 0.00 -> 36.9 mm, vias 0 -> 4
- net /BASE_R2: track 0.00 -> 32.7 mm, vias 0 -> 4
- net /USART1_DE: track 0.00 -> 30.6 mm, vias 0 -> 2
- net /R5: track 16.2 -> 44.0 mm, vias 2 -> 3
- net /USART1_TX: track 0.00 -> 25.2 mm, vias 0 -> 2
- net RESET: track 0.00 -> 23.2 mm, vias 0 -> 2
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- added copper zone on B.Cu, net GND
- added copper zone on F.Cu, net GND
Other:
- outline, holes or cut-outs redrawn
- board text added: "3- RS232 TX 4,5- GND 6- RS232 RX 7- RS485 A 8- RS485 B"
- board text added: "3V3"
- board text added: "BOOT"
- board text added: "RESET"
- board text added: "SWCLK"
- board text added: "SWDIO"
